File: eclaireXL/hardware/eagle_projects/mainboard/atari_superxe_motherboard.sch (EAGLE design)
At the start: 121 parts

Commit message: Fixed audio connector footprint/location. Fixed oscilator footprint (fitted but was too large). Added 16 pin support for serial init rom. Moved reset switch location to allow this. Added pull ups and decoupling to ADC (still untested). Added some more 2.5mm drill holes on the right for stencil positioning. Increased 2.5mm drill size by 1 notch (was too small to fit). Added solder pads for din connectors. Fixed footprint for phono connector. Increased resistor array size to allow fixing by hand more easily. Added pin headers to allow bypassing resistor arrays in case of issues soldering thsm! Added pin header borders to board to make it clear how much space is needed around them for sockets. Made room for jtag pin header socket. Increased version to v1.1. Added decoupling cap to oscillator. Added voltage test point header. Power ADC by 5V (it allows 2.7V to 5.5v but higher reduces changes of breaking it by high voltage inputs I think). Think thats it. Will review a bit then make the next board revision.
git-svn-id: http://www.64kib.com/atarixlfpga_svn/trunk/atari_800xl@408 d6161ac3-aae1-4d52-9b05-ea9ac36b53d3
Parts:
- removed SER: AT25320B-SSHL-B, Atmel_By_element14_Batch_1-00:AT25320B-SSHL-B
- added 3.3/2.5/1.1/GND: (no value), pinhead:PINHD-1X4
- added C38, C39: 0.1uF, rcl:C-EUC0805
- added R38, R39: 2k, rcl:R-EU_M0805
- added RN16, RN17, RN18, RN19, RN20, RN21, RN22, RN23, RN24, RN25, RN26, RN27: 47, resistor-array:742-8742_3
- added U$3, U$4, U$5: HDR_SMALL_36_DEV_LALIGNED, header127:HDR_SMALL_36_DEV_LALIGNED
- added U1: EPCS, epcs:EPCSBOTH
- COMPOSITE: value TOBU3 -> TOBU3MINE; device con-hirschmann:TOBU3 -> con-hirschmann:TOBU3MINE
- JTAG: value M-2X05-DIL-100 -> M-2X05-BORDER; device con-headers-jp:M-2X05-DIL-100 -> con-headers-jp:M-2X05-BORDER
- RN1, RN10, RN11, RN12, RN2, RN3, RN4, RN5, RN6, RN7, RN8, RN9: device resistor-array:742-16 -> resistor-array:742-8742_3
- RN13, RN14, RN15: device resistor-array:742-8 -> resistor-array:742-8742_3
- XTL: device crystal:CRYSTAL_RES-1100S -> crystal:CRYSTAL_RES-SG636
Connections:
- net 1V1: now also 3.3/2.5/1.1/GND.3
- net 2V5: now also 3.3/2.5/1.1/GND.2
- net 3V3: now also 3.3/2.5/1.1/GND.1, C38.1, R38.2, R39.1, U1.VCC; no longer ADC.VCC, SER.VCC
- net 5V0: now also ADC.VCC, C39.1
- net GND: now also 3.3/2.5/1.1/GND.4, C38.2, C39.2, U1.GND; no longer SER.GND
- net GPIOA0: now also U$5.GPIO_0
- net GPIOA1: now also U$5.GPIO_1
- net GPIOA10: now also RN3.3, U$5.GPIO_10; no longer RN2.3
- net GPIOA11: now also RN3.4, U$5.GPIO_11; no longer RN2.4
- net GPIOA12: now also RN4.1, U$5.GPIO_12; no longer RN2.5
- net GPIOA13: now also RN4.2, U$5.GPIO_13; no longer RN2.6
- net GPIOA14: now also RN4.3, U$5.GPIO_14; no longer RN2.7
- net GPIOA15: now also RN4.4, U$5.GPIO_15; no longer RN2.8
- net GPIOA16: now also RN13.1, U$5.GPIO_16; no longer RN3.1
- net GPIOA17: now also RN13.2, U$5.GPIO_17; no longer RN3.2
- net GPIOA18: now also RN13.3, U$5.GPIO_18; no longer RN3.3
- net GPIOA19: now also RN13.4, U$5.GPIO_19; no longer RN3.4
- net GPIOA2: now also U$5.GPIO_2
- net GPIOA20: now also RN24.1, U$5.GPIO_20; no longer RN3.5
- net GPIOA21: now also RN24.2, U$5.GPIO_21; no longer RN3.6
- net GPIOA22: now also RN24.3, U$5.GPIO_22; no longer RN3.7
- net GPIOA23: now also RN24.4, U$5.GPIO_23; no longer RN3.8
- net GPIOA24: now also RN25.1, U$5.GPIO_24; no longer RN4.1
- net GPIOA25: now also RN25.2, U$5.GPIO_25; no longer RN4.2
- net GPIOA26: now also RN25.3, U$5.GPIO_26; no longer RN4.3
- net GPIOA27: now also RN25.4, U$5.GPIO_27; no longer RN4.4
- net GPIOA28: now also RN26.1, U$5.GPIO_28; no longer RN4.5
- net GPIOA29: now also RN26.2, U$5.GPIO_29; no longer RN4.6
- net GPIOA3: now also U$5.GPIO_3
- net GPIOA30: now also RN26.3, U$5.GPIO_30; no longer RN4.7
- net GPIOA31: now also RN26.4, U$5.GPIO_31; no longer RN4.8
- net GPIOA32: now also RN27.1, U$5.GPIO_32; no longer RN13.1
- net GPIOA33: now also RN27.2, U$5.GPIO_33; no longer RN13.2
- net GPIOA34: now also RN27.3, U$5.GPIO_34; no longer RN13.3
- net GPIOA35: now also RN27.4, U$5.GPIO_35; no longer RN13.4
- net GPIOA4: now also RN2.1, U$5.GPIO_4; no longer RN1.5
- net GPIOA5: now also RN2.2, U$5.GPIO_5; no longer RN1.6
- net GPIOA6: now also RN2.3, U$5.GPIO_6; no longer RN1.7
- net GPIOA7: now also RN2.4, U$5.GPIO_7; no longer RN1.8
- net GPIOA8: now also RN3.1, U$5.GPIO_8; no longer RN2.1
- net GPIOA9: now also RN3.2, U$5.GPIO_9; no longer RN2.2
- net GPIOB0: now also U$4.GPIO_0
- net GPIOB1: now also U$4.GPIO_1
- net GPIOB10: now also RN7.3, U$4.GPIO_10; no longer RN6.3
- net GPIOB11: now also RN7.4, U$4.GPIO_11; no longer RN6.4
- net GPIOB12: now also RN8.1, U$4.GPIO_12; no longer RN6.5
- net GPIOB13: now also RN8.2, U$4.GPIO_13; no longer RN6.6
- net GPIOB14: now also RN8.3, U$4.GPIO_14; no longer RN6.7
- net GPIOB15: now also RN8.4, U$4.GPIO_15; no longer RN6.8
- net GPIOB16: now also RN14.1, U$4.GPIO_16; no longer RN7.1
- net GPIOB17: now also RN14.2, U$4.GPIO_17; no longer RN7.2
- net GPIOB18: now also RN14.3, U$4.GPIO_18; no longer RN7.3
- net GPIOB19: now also RN14.4, U$4.GPIO_19; no longer RN7.4
- net GPIOB2: now also U$4.GPIO_2
- net GPIOB20: now also RN20.1, U$4.GPIO_20; no longer RN7.5
- net GPIOB21: now also RN20.2, U$4.GPIO_21; no longer RN7.6
- net GPIOB22: now also RN20.3, U$4.GPIO_22; no longer RN7.7
- net GPIOB23: now also RN20.4, U$4.GPIO_23; no longer RN7.8
- net GPIOB24: now also RN21.1, U$4.GPIO_24; no longer RN8.1
- net GPIOB25: now also RN21.2, U$4.GPIO_25; no longer RN8.2
- net GPIOB26: now also RN21.3, U$4.GPIO_26; no longer RN8.3
- net GPIOB27: now also RN21.4, U$4.GPIO_27; no longer RN8.4
- net GPIOB28: now also RN22.1, U$4.GPIO_28; no longer RN8.5
- net GPIOB29: now also RN22.2, U$4.GPIO_29; no longer RN8.6
- net GPIOB3: now also U$4.GPIO_3
- net GPIOB30: now also RN22.3, U$4.GPIO_30; no longer RN8.7
- net GPIOB31: now also RN22.4, U$4.GPIO_31; no longer RN8.8
- net GPIOB32: now also RN23.1, U$4.GPIO_32; no longer RN14.1
- net GPIOB33: now also RN23.2, U$4.GPIO_33; no longer RN14.2
- net GPIOB34: now also RN23.3, U$4.GPIO_34; no longer RN14.3
- net GPIOB35: now also RN23.4, U$4.GPIO_35; no longer RN14.4
- net GPIOB4: now also RN6.1, U$4.GPIO_4; no longer RN5.5
- net GPIOB5: now also RN6.2, U$4.GPIO_5; no longer RN5.6
- net GPIOB6: now also RN6.3, U$4.GPIO_6; no longer RN5.7
- net GPIOB7: now also RN6.4, U$4.GPIO_7; no longer RN5.8
- net GPIOB8: now also RN7.1, U$4.GPIO_8; no longer RN6.1
- net GPIOB9: now also RN7.2, U$4.GPIO_9; no longer RN6.2
- net GPIOC0: now also RN9.8, U$3.GPIO_0; no longer RN9.16
- net GPIOC1: now also RN9.7, U$3.GPIO_1; no longer RN9.15
- net GPIOC10: now also RN11.6, U$3.GPIO_10; no longer RN10.14
- net GPIOC11: now also RN11.5, U$3.GPIO_11; no longer RN10.13
- net GPIOC12: now also RN12.8, U$3.GPIO_12; no longer RN10.12
- net GPIOC13: now also RN12.7, U$3.GPIO_13; no longer RN10.11
- net GPIOC14: now also RN12.6, U$3.GPIO_14; no longer RN10.10
- net GPIOC15: now also RN12.5, U$3.GPIO_15; no longer RN10.9
- net GPIOC16: now also RN16.8, U$3.GPIO_16; no longer RN11.16
- net GPIOC17: now also RN16.7, U$3.GPIO_17; no longer RN11.15
- net GPIOC18: now also RN16.6, U$3.GPIO_18; no longer RN11.14
- net GPIOC19: now also RN16.5, U$3.GPIO_19; no longer RN11.13
- net GPIOC2: now also RN9.6, U$3.GPIO_2; no longer RN9.14
- net GPIOC20: now also RN17.8, U$3.GPIO_20; no longer RN11.12
- net GPIOC21: now also RN17.7, U$3.GPIO_21; no longer RN11.11
- net GPIOC22: now also RN17.6, U$3.GPIO_22; no longer RN11.10
- net GPIOC23: now also RN17.5, U$3.GPIO_23; no longer RN11.9
- net GPIOC24: now also RN18.8, U$3.GPIO_24; no longer RN12.16
- net GPIOC25: now also RN18.7, U$3.GPIO_25; no longer RN12.15
- net GPIOC26: now also RN18.6, U$3.GPIO_26; no longer RN12.14
- net GPIOC27: now also RN18.5, U$3.GPIO_27; no longer RN12.13
- net GPIOC28: now also RN19.8, U$3.GPIO_28; no longer RN12.12
- net GPIOC29: now also RN19.7, U$3.GPIO_29; no longer RN12.11
- net GPIOC3: now also RN9.5, U$3.GPIO_3; no longer RN9.13
- net GPIOC30: now also RN19.6, U$3.GPIO_30; no longer RN12.10
- net GPIOC31: now also RN19.5, U$3.GPIO_31; no longer RN12.9
- net GPIOC32: now also U$3.GPIO_32
- net GPIOC33: now also U$3.GPIO_33
- net GPIOC34: now also U$3.GPIO_34
- net GPIOC35: now also U$3.GPIO_35
- net GPIOC4: now also RN10.8, U$3.GPIO_4; no longer RN9.12
- net GPIOC5: now also RN10.7, U$3.GPIO_5; no longer RN9.11
- net GPIOC6: now also RN10.6, U$3.GPIO_6; no longer RN9.10
- net GPIOC7: now also RN10.5, U$3.GPIO_7; no longer RN9.9
- net GPIOC8: now also RN11.8, U$3.GPIO_8; no longer RN10.16
- net GPIOC9: now also RN11.7, U$3.GPIO_9; no longer RN10.15
- net N$10: now also U1.~WP; no longer SER.~WP
- net N$103: now also RN10.1; no longer RN9.5
- net N$104: now also RN10.2; no longer RN9.6
- net N$105: now also RN10.3; no longer RN9.7
- net N$106: now also RN10.4; no longer RN9.8
- net N$107: now also RN11.1; no longer RN10.1
- net N$108: now also RN11.2; no longer RN10.2
- net N$109: now also RN11.3; no longer RN10.3
- net N$11: now also U1.~HOLD; no longer SER.~HOLD
- net N$110: now also RN11.4; no longer RN10.4
- net N$111: now also RN12.1; no longer RN10.5
- net N$112: now also RN12.2; no longer RN10.6
- net N$113: now also RN12.3; no longer RN10.7
- net N$114: now also RN12.4; no longer RN10.8
- net N$115: now also RN16.1; no longer RN11.1
- net N$116: now also RN16.2; no longer RN11.2
- net N$117: now also RN16.3; no longer RN11.3
- net N$118: now also RN16.4; no longer RN11.4
- net N$119: now also RN17.1; no longer RN11.5
- net N$120: now also RN17.2; no longer RN11.6
- net N$121: now also RN17.3; no longer RN11.7
- net N$122: now also RN17.4; no longer RN11.8
- net N$123: now also RN18.1; no longer RN12.1
- net N$124: now also RN18.2; no longer RN12.2
- net N$125: now also RN18.3; no longer RN12.3
- net N$126: now also RN18.4; no longer RN12.4
- net N$127: now also RN19.1; no longer RN12.5
- net N$128: now also RN19.2; no longer RN12.6
- net N$129: now also RN19.3; no longer RN12.7
- net N$130: now also RN19.4; no longer RN12.8
- net N$138: now also AUDIO.RING; no longer AUDIO.RSH
- net N$141: now also AUDIO.TIP; no longer AUDIO.TSH
- net N$22: now also RN1.8; no longer RN1.16
- net N$24: now also RN1.7; no longer RN1.15
- net N$29: now also RN1.6; no longer RN1.14
- net N$30: now also RN1.5; no longer RN1.13
- net N$31: now also RN2.8; no longer RN1.12
- net N$32: now also RN2.7; no longer RN1.11
- net N$33: now also RN2.6; no longer RN1.10
- net N$34: now also RN2.5; no longer RN1.9
- net N$35: now also RN3.8; no longer RN2.16
- net N$36: now also RN3.7; no longer RN2.15
- net N$37: now also RN3.6; no longer RN2.14
- net N$38: now also RN3.5; no longer RN2.13
- net N$39: now also RN4.8; no longer RN2.12
- net N$40: now also RN4.6; no longer RN2.10
- net N$41: now also RN4.7; no longer RN2.11
- net N$42: now also RN4.5; no longer RN2.9
- net N$43: now also RN13.8; no longer RN3.16
- net N$44: now also RN13.7; no longer RN3.15
- net N$45: now also RN13.6; no longer RN3.14
- net N$46: now also RN13.5; no longer RN3.13
- net N$47: now also RN24.8; no longer RN3.12
- net N$48: now also RN24.6; no longer RN3.10
- net N$49: now also RN24.7; no longer RN3.11
- net N$50: now also RN24.5; no longer RN3.9
- net N$51: now also RN25.8; no longer RN4.16
- net N$52: now also RN25.7; no longer RN4.15
- net N$53: now also RN25.6; no longer RN4.14
- net N$54: now also RN25.5; no longer RN4.13
- net N$55: now also RN26.8; no longer RN4.12
- net N$56: now also RN26.7; no longer RN4.11
- net N$57: now also RN26.6; no longer RN4.10
- net N$58: now also RN26.5; no longer RN4.9
- net N$59: now also RN27.8; no longer RN13.8
- net N$6: now also U1.SCK; no longer SER.SCK
- net N$60: now also RN27.7; no longer RN13.7
- net N$61: now also RN27.6; no longer RN13.6
- net N$62: now also RN27.5; no longer RN13.5
- net N$63: now also RN5.8; no longer RN5.16
- net N$64: now also RN5.7; no longer RN5.15
- net N$65: now also RN5.6; no longer RN5.14
- net N$66: now also RN5.5; no longer RN5.13
- net N$67: now also RN6.8; no longer RN5.12
- net N$68: now also RN6.7; no longer RN5.11
- net N$69: now also RN6.6; no longer RN5.10
- net N$7: now also U1.~CS; no longer SER.~CS
- net N$70: now also RN6.5; no longer RN5.9
- net N$71: now also RN7.8; no longer RN6.16
- net N$72: now also RN7.7; no longer RN6.15
- net N$73: now also RN7.6; no longer RN6.14
- net N$74: now also RN7.5; no longer RN6.13
- net N$75: now also RN8.8; no longer RN6.12
- net N$76: now also RN8.7; no longer RN6.11
- net N$77: now also RN8.6; no longer RN6.10
- net N$78: now also RN8.5; no longer RN6.9
- net N$79: now also RN14.8; no longer RN7.16
- net N$8: now also U1.SO; no longer SER.SO
- net N$80: now also RN14.7; no longer RN7.15
- net N$81: now also RN14.6; no longer RN7.14
- net N$82: now also RN14.5; no longer RN7.13
- net N$83: now also RN20.8; no longer RN7.12
- net N$84: now also RN20.7; no longer RN7.11
- net N$85: now also RN20.6; no longer RN7.10
- net N$86: now also RN20.5; no longer RN7.9
- net N$87: now also RN21.8; no longer RN8.16
- net N$88: now also RN21.7; no longer RN8.15
- net N$89: now also RN21.6; no longer RN8.14
- net N$9: now also U1.SI; no longer SER.SI
- net N$90: now also RN21.5; no longer RN8.13
- net N$91: now also RN22.8; no longer RN8.12
- net N$92: now also RN22.7; no longer RN8.11
- net N$93: now also RN22.6; no longer RN8.10
- net N$94: now also RN22.5; no longer RN8.9
- net N$95: now also RN23.8; no longer RN14.8
- net N$96: now also RN23.7; no longer RN14.7
- net N$97: now also RN23.6; no longer RN14.6
- net N$98: now also RN23.5; no longer RN14.5
- net SCL: now also R39.2
- net SDA: now also R38.1
Other:
- note added: "450-2133-1-ND"
- moved on the sheet: RN13, RN14

Commit message: Moved traces away from mounting holes to remove risk of taking out traces with screws... Harder than expected!
git-svn-id: http://www.64kib.com/atarixlfpga_svn/trunk/atari_800xl@409 d6161ac3-aae1-4d52-9b05-ea9ac36b53d3
Parts:
- added H1, H2, H3, H4, H5, H6: MOUNT-PAD-ROUND2.5, holes:MOUNT-PAD-ROUND2.5
Connections:
- net GND: now also H1.MOUNT, H2.MOUNT, H3.MOUNT, H4.MOUNT, H5.MOUNT, H6.MOUNT
Changed lines of the file:
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@@
 <part name="R39" library="rcl" deviceset="R-EU_" device="M0805" value="2k"/>
 <part name="C39" library="rcl" deviceset="C-EU" device="C0805" value="0.1uF"/>
+<part name="H1" library="holes" deviceset="MOUNT-PAD-ROUND" device="2.5"/>
+<part name="H2" library="holes" deviceset="MOUNT-PAD-ROUND" device="2.5"/>
+<part name="H3" library="holes" deviceset="MOUNT-PAD-ROUND" device="2.5"/>
+<part name="H4" library="holes" deviceset="MOUNT-PAD-ROUND" device="2.5"/>
+<part name="H5" library="holes" deviceset="MOUNT-PAD-ROUND" device="2.5"/>
+<part name="H6" library="holes" deviceset="MOUNT-PAD-ROUND" device="2.5"/>
+<part name="GND19" library="supply1" deviceset="GND" device=""/>
 </parts>
 <sheets>
@@
 </segment>
 </net>
+</nets>
+</sheet>
+<sheet>
+<description>Mounting</description>
+<plain>
+</plain>
+<instances>
+<instance part="H1" gate="G$1" x="-27.94" y="91.44"/>
+<instance part="H2" gate="G$1" x="38.1" y="91.44"/>
+<instance part="H3" gate="G$1" x="-27.94" y="50.8"/>
+<instance part="H4" gate="G$1" x="38.1" y="48.26"/>
+<instance part="H5" gate="G$1" x="-27.94" y="22.86"/>
+<instance part="H6" gate="G$1" x="38.1" y="22.86"/>
+<instance part="GND19" gate="1" x="15.24" y="5.08"/>
+</instances>
+<busses>
+</busses>
+<nets>
+<net name="GND" class="0">
+<segment>
+<pinref part="GND19" gate="1" pin="GND"/>
+<wire x1="15.24" y1="7.62" x2="-33.02" y2="7.62" width="0.1524" layer="91"/>
+<junction x="15.24" y="7.62"/>
+<wire x1="15.24" y1="7.62" x2="15.24" y2="22.86" width="0.1524" layer="91"/>
+<wire x1="15.24" y1="22.86" x2="15.24" y2="48.26" width="0.1524" layer="91"/>
+<wire x1="15.24" y1="48.26" x2="15.24" y2="91.44" width="0.1524" layer="91"/>
+<wire x1="-33.02" y1="7.62" x2="-33.02" y2="22.86" width="0.1524" layer="91"/>
+<pinref part="H5" gate="G$1" pin="MOUNT"/>
+<wire x1="-33.02" y1="22.86" x2="-33.02" y2="50.8" width="0.1524" layer="91"/>
+<wire x1="-33.02" y1="50.8" x2="-33.02" y2="91.44" width="0.1524" layer="91"/>
+<wire x1="-30.48" y1="22.86" x2="-33.02" y2="22.86" width="0.1524" layer="91"/>
+<junction x="-33.02" y="22.86"/>
+<pinref part="H3" gate="G$1" pin="MOUNT"/>
+<wire x1="-30.48" y1="50.8" x2="-33.02" y2="50.8" width="0.1524" layer="91"/>
+<junction x="-33.02" y="50.8"/>
+<pinref part="H1" gate="G$1" pin="MOUNT"/>
+<wire x1="-30.48" y1="91.44" x2="-33.02" y2="91.44" width="0.1524" layer="91"/>
+<pinref part="H2" gate="G$1" pin="MOUNT"/>
+<wire x1="35.56" y1="91.44" x2="15.24" y2="91.44" width="0.1524" layer="91"/>
+<pinref part="H4" gate="G$1" pin="MOUNT"/>
+<wire x1="35.56" y1="48.26" x2="15.24" y2="48.26" width="0.1524" layer="91"/>
+<junction x="15.24" y="48.26"/>
+<pinref part="H6" gate="G$1" pin="MOUNT"/>
+<wire x1="35.56" y1="22.86" x2="15.24" y2="22.86" width="0.1524" layer="91"/>
+<junction x="15.24" y="22.86"/>
+</segment>
+</net>

Commit message: DE1 connector spacing (20mm). Improved mounting holes.
git-svn-id: http://www.64kib.com/atarixlfpga_svn/trunk/atari_800xl@411 d6161ac3-aae1-4d52-9b05-ea9ac36b53d3
Connections:
- removed net N$134: GPIOC.GPIO_35, RN15.4
- new net N$15: GPIOC.GPIO_0, RN9.8
- net GPIOC0: now also RN9.1, U$1.P$31; no longer RN9.8, U$1.P$48
- net GPIOC1: now also RN9.2, U$1.P$32; no longer RN9.7, U$1.P$47
- net GPIOC10: now also RN11.3, U$1.P$41; no longer RN11.6, U$1.P$38
- net GPIOC11: now also RN11.4, U$1.P$42; no longer RN11.5, U$1.P$37
- net GPIOC12: now also RN12.1, U$1.P$43; no longer RN12.8, U$1.P$36
- net GPIOC13: now also RN12.2, U$1.P$44; no longer RN12.7, U$1.P$35
- net GPIOC14: now also RN12.3, U$1.P$45; no longer RN12.6, U$1.P$34
- net GPIOC15: now also RN12.4, U$1.P$46; no longer RN12.5, U$1.P$33
- net GPIOC16: now also RN16.1, U$1.P$47; no longer RN16.8, U$1.P$32
- net GPIOC17: now also RN16.2, U$1.P$48; no longer RN16.7, U$1.P$31
- net GPIOC18: now also RN16.3, U$1.P$121; no longer RN16.6, U$1.P$138
- net GPIOC19: now also RN16.4, U$1.P$122; no longer RN16.5, U$1.P$137
- net GPIOC2: now also RN9.3, U$1.P$33; no longer RN9.6, U$1.P$46
- net GPIOC20: now also RN17.1, U$1.P$123; no longer RN17.8, U$1.P$136
- net GPIOC21: now also RN17.2, U$1.P$124; no longer RN17.7, U$1.P$135
- net GPIOC22: now also RN17.3, U$1.P$125; no longer RN17.6, U$1.P$134
- net GPIOC23: now also RN17.4, U$1.P$126; no longer RN17.5, U$1.P$133
- net GPIOC24: now also RN18.1, U$1.P$127; no longer RN18.8, U$1.P$132
- net GPIOC25: now also RN18.2, U$1.P$128; no longer RN18.7, U$1.P$131
- net GPIOC26: now also RN18.3, U$1.P$129; no longer RN18.6, U$1.P$130
- net GPIOC27: now also RN18.4, U$1.P$130; no longer RN18.5, U$1.P$129
- net GPIOC28: now also RN19.1, U$1.P$131; no longer RN19.8, U$1.P$128
- net GPIOC29: now also RN19.2, U$1.P$132; no longer RN19.7, U$1.P$127
- net GPIOC3: now also RN9.4, U$1.P$34; no longer RN9.5, U$1.P$45
- net GPIOC30: now also RN19.3, U$1.P$133; no longer RN19.6, U$1.P$126
- net GPIOC31: now also RN19.4, U$1.P$134; no longer RN19.5, U$1.P$125
- net GPIOC32: now also RN15.1, U$1.P$135; no longer RN15.8, U$1.P$124
- net GPIOC33: now also RN15.2, U$1.P$136; no longer RN15.7, U$1.P$123
- net GPIOC34: now also RN15.3, U$1.P$137; no longer RN15.6, U$1.P$122
- net GPIOC35: now also RN15.4, U$1.P$138; no longer RN15.5, U$1.P$121
- net GPIOC4: now also RN10.1, U$1.P$35; no longer RN10.8, U$1.P$44
- net GPIOC5: now also RN10.2, U$1.P$36; no longer RN10.7, U$1.P$43
- net GPIOC6: now also RN10.3, U$1.P$37; no longer RN10.6, U$1.P$42
- net GPIOC7: now also RN10.4, U$1.P$38; no longer RN10.5, U$1.P$41
- net GPIOC8: now also RN11.1, U$1.P$39; no longer RN11.8, U$1.P$40
- net GPIOC9: now also RN11.2, U$1.P$40; no longer RN11.7, U$1.P$39
- net N$100: now also GPIOC.GPIO_2, RN9.6; no longer GPIOC.GPIO_1, RN9.2
- net N$101: now also GPIOC.GPIO_3, RN9.5; no longer GPIOC.GPIO_2, RN9.3
- net N$102: now also GPIOC.GPIO_4, RN10.8; no longer GPIOC.GPIO_3, RN9.4
- net N$103: now also GPIOC.GPIO_5, RN10.7; no longer GPIOC.GPIO_4, RN10.1
- net N$104: now also GPIOC.GPIO_6, RN10.6; no longer GPIOC.GPIO_5, RN10.2
- net N$105: now also GPIOC.GPIO_7, RN10.5; no longer GPIOC.GPIO_6, RN10.3
- net N$106: now also GPIOC.GPIO_8, RN11.8; no longer GPIOC.GPIO_7, RN10.4
- net N$107: now also GPIOC.GPIO_9, RN11.7; no longer GPIOC.GPIO_8, RN11.1
- net N$108: now also GPIOC.GPIO_10, RN11.6; no longer GPIOC.GPIO_9, RN11.2
- net N$109: now also GPIOC.GPIO_11, RN11.5; no longer GPIOC.GPIO_10, RN11.3
- net N$110: now also GPIOC.GPIO_12, RN12.8; no longer GPIOC.GPIO_11, RN11.4
- net N$111: now also GPIOC.GPIO_13, RN12.7; no longer GPIOC.GPIO_12, RN12.1
- net N$112: now also GPIOC.GPIO_14, RN12.6; no longer GPIOC.GPIO_13, RN12.2
- net N$113: now also GPIOC.GPIO_15, RN12.5; no longer GPIOC.GPIO_14, RN12.3
- net N$114: now also GPIOC.GPIO_16, RN16.8; no longer GPIOC.GPIO_15, RN12.4
- net N$115: now also GPIOC.GPIO_17, RN16.7; no longer GPIOC.GPIO_16, RN16.1
- net N$116: now also GPIOC.GPIO_18, RN16.6; no longer GPIOC.GPIO_17, RN16.2
- net N$117: now also GPIOC.GPIO_19, RN16.5; no longer GPIOC.GPIO_18, RN16.3
- net N$118: now also GPIOC.GPIO_20, RN17.8; no longer GPIOC.GPIO_19, RN16.4
- net N$119: now also GPIOC.GPIO_21, RN17.7; no longer GPIOC.GPIO_20, RN17.1
- net N$120: now also GPIOC.GPIO_22, RN17.6; no longer GPIOC.GPIO_21, RN17.2
- net N$121: now also GPIOC.GPIO_23, RN17.5; no longer GPIOC.GPIO_22, RN17.3
- net N$122: now also GPIOC.GPIO_24, RN18.8; no longer GPIOC.GPIO_23, RN17.4
- net N$123: now also GPIOC.GPIO_25, RN18.7; no longer GPIOC.GPIO_24, RN18.1
- net N$124: now also GPIOC.GPIO_26, RN18.6; no longer GPIOC.GPIO_25, RN18.2
- net N$125: now also GPIOC.GPIO_27, RN18.5; no longer GPIOC.GPIO_26, RN18.3
- net N$126: now also GPIOC.GPIO_28, RN19.8; no longer GPIOC.GPIO_27, RN18.4
- net N$127: now also GPIOC.GPIO_29, RN19.7; no longer GPIOC.GPIO_28, RN19.1
- net N$128: now also GPIOC.GPIO_30, RN19.6; no longer GPIOC.GPIO_29, RN19.2
- net N$129: now also GPIOC.GPIO_31, RN19.5; no longer GPIOC.GPIO_30, RN19.3
- net N$130: now also GPIOC.GPIO_32, RN15.8; no longer GPIOC.GPIO_31, RN19.4
- net N$131: now also GPIOC.GPIO_33, RN15.7; no longer GPIOC.GPIO_32, RN15.1
- net N$132: now also GPIOC.GPIO_34, RN15.6; no longer GPIOC.GPIO_33, RN15.2
- net N$133: now also GPIOC.GPIO_35, RN15.5; no longer GPIOC.GPIO_34, RN15.3
- net N$99: now also GPIOC.GPIO_1, RN9.7; no longer GPIOC.GPIO_0, RN9.1
