File: eclaireXL/hardware/eagle_projects/mainboard/atari_superxe_motherboard.sch (EAGLE design)
At the start: 147 parts, among them U1 EPCS

Commit message: Moved video ports to the back (painful!!). Added rocker switch on left for power.
git-svn-id: http://www.64kib.com/atarixlfpga_svn/trunk/atari_800xl@424 d6161ac3-aae1-4d52-9b05-ea9ac36b53d3
Parts:
- added H7: MOUNT-PAD-ROUND2.5, holes:MOUNT-PAD-ROUND2.5
- POW: value 450302014072 -> 450302014072ROCKER; device Eagle_Wuerth_Elektronik_Switch_rev15b:450302014072 -> Eagle_Wuerth_Elektronik_Switch_rev15b:450302014072ROCKER
- U$2: value SDMMC06132 -> SDMMCHALFHEIGHT; device adafruit:SDMMC06132 -> adafruit:SDMMCHALFHEIGHT
Connections:
- net 5V0: now also POW.2; no longer POW.1
- net GND: now also H7.MOUNT
- net N$139: now also POW.1; no longer POW.3
Changed lines of the file:
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@@
 <grid distance="0.1" unitdist="inch" unit="inch" style="lines" multiple="1" display="no" altdistance="0.01" altunitdist="inch" altunit="inch"/>
 <layers>
-<layer number="1" name="Top" color="4" fill="1" visible="no" active="no"/>
-<layer number="2" name="Route2" color="1" fill="3" visible="no" active="no"/>
-<layer number="3" name="Route3" color="4" fill="3" visible="no" active="no"/>
-<layer number="14" name="Route14" color="1" fill="6" visible="no" active="no"/>
-<layer number="15" name="Route15" color="4" fill="6" visible="no" active="no"/>
-<layer number="16" name="Bottom" color="1" fill="1" visible="no" active="no"/>
-<layer number="17" name="Pads" color="2" fill="1" visible="no" active="no"/>
-<layer number="18" name="Vias" color="2" fill="1" visible="no" active="no"/>
-<layer number="19" name="Unrouted" color="6" fill="1" visible="no" active="no"/>
-<layer number="20" name="Dimension" color="15" fill="1" visible="no" active="no"/>
-<layer number="21" name="tPlace" color="7" fill="1" visible="no" active="no"/>
-<layer number="22" name="bPlace" color="7" fill="1" visible="no" active="no"/>
-<layer number="23" name="tOrigins" color="15" fill="1" visible="no" active="no"/>
-<layer number="24" name="bOrigins" color="15" fill="1" visible="no" active="no"/>
-<layer number="25" name="tNames" color="7" fill="1" visible="no" active="no"/>
-<layer number="26" name="bNames" color="7" fill="1" visible="no" active="no"/>
-<layer number="27" name="tValues" color="7" fill="1" visible="no" active="no"/>
-<layer number="28" name="bValues" color="7" fill="1" visible="no" active="no"/>
+<layer number="1" name="Top" color="4" fill="1" visible="yes" active="no"/>
+<layer number="2" name="Route2" color="1" fill="3" visible="yes" active="no"/>
+<layer number="3" name="Route3" color="4" fill="3" visible="yes" active="no"/>
+<layer number="14" name="Route14" color="1" fill="6" visible="yes" active="no"/>
+<layer number="15" name="Route15" color="4" fill="6" visible="yes" active="no"/>
+<layer number="16" name="Bottom" color="1" fill="1" visible="yes" active="no"/>
+<layer number="17" name="Pads" color="2" fill="1" visible="yes" active="no"/>
+<layer number="18" name="Vias" color="2" fill="1" visible="yes" active="no"/>
+<layer number="19" name="Unrouted" color="6" fill="1" visible="yes" active="no"/>
+<layer number="20" name="Dimension" color="15" fill="1" visible="yes" active="no"/>
+<layer number="21" name="tPlace" color="7" fill="1" visible="yes" active="no"/>
+<layer number="22" name="bPlace" color="7" fill="1" visible="yes" active="no"/>
+<layer number="23" name="tOrigins" color="15" fill="1" visible="yes" active="no"/>
+<layer number="24" name="bOrigins" color="15" fill="1" visible="yes" active="no"/>
+<layer number="25" name="tNames" color="7" fill="1" visible="yes" active="no"/>
+<layer number="26" name="bNames" color="7" fill="1" visible="yes" active="no"/>
+<layer number="27" name="tValues" color="7" fill="1" visible="yes" active="no"/>
+<layer number="28" name="bValues" color="7" fill="1" visible="yes" active="no"/>
 <layer number="29" name="tStop" color="7" fill="3" visible="no" active="no"/>
 <layer number="30" name="bStop" color="7" fill="6" visible="no" active="no"/>
@@
 <layer number="35" name="tGlue" color="7" fill="4" visible="no" active="no"/>
 <layer number="36" name="bGlue" color="7" fill="5" visible="no" active="no"/>
-<layer number="37" name="tTest" color="7" fill="1" visible="no" active="no"/>
-<layer number="38" name="bTest" color="7" fill="1" visible="no" active="no"/>
+<layer number="37" name="tTest" color="7" fill="1" visible="yes" active="no"/>
+<layer number="38" name="bTest" color="7" fill="1" visible="yes" active="no"/>
 <layer number="39" name="tKeepout" color="4" fill="11" visible="no" active="no"/>
 <layer number="40" name="bKeepout" color="1" fill="11" visible="no" active="no"/>
@@
 <layer number="44" name="Drills" color="7" fill="1" visible="no" active="no"/>
 <layer number="45" name="Holes" color="7" fill="1" visible="no" active="no"/>
-<layer number="46" name="Milling" color="3" fill="1" visible="no" active="no"/>
-<layer number="47" name="Measures" color="7" fill="1" visible="no" active="no"/>
-<layer number="48" name="Document" color="7" fill="1" visible="no" active="no"/>
-<layer number="49" name="Reference" color="7" fill="1" visible="no" active="no"/>
-<layer number="50" name="dxf" color="7" fill="1" visible="no" active="no"/>
-<layer number="51" name="tDocu" color="7" fill="1" visible="no" active="no"/>
-<layer number="52" name="bDocu" color="7" fill="1" visible="no" active="no"/>
-<layer number="53" name="tGND_GNDA" color="7" fill="9" visible="no" active="no"/>
-<layer number="54" name="bGND_GNDA" color="1" fill="9" visible="no" active="no"/>
-<layer number="56" name="wert" color="7" fill="1" visible="no" active="no"/>
-<layer number="57" name="tCAD" color="7" fill="1" visible="no" active="no"/>
-<layer number="58" name="bCAD" color="11" fill="1" visible="no" active="no"/>
+<layer number="46" name="Milling" color="3" fill="1" visible="yes" active="no"/>
+<layer number="47" name="Measures" color="7" fill="1" visible="yes" active="no"/>
+<layer number="48" name="Document" color="7" fill="1" visible="yes" active="no"/>
+<layer number="49" name="Reference" color="7" fill="1" visible="yes" active="no"/>
+<layer number="50" name="dxf" color="7" fill="1" visible="yes" active="no"/>
+<layer number="51" name="tDocu" color="7" fill="1" visible="yes" active="no"/>
+<layer number="52" name="bDocu" color="7" fill="1" visible="yes" active="no"/>
+<layer number="53" name="tGND_GNDA" color="7" fill="9" visible="yes" active="no"/>
+<layer number="54" name="bGND_GNDA" color="1" fill="9" visible="yes" active="no"/>
+<layer number="56" name="wert" color="7" fill="1" visible="yes" active="no"/>
+<layer number="57" name="tCAD" color="7" fill="1" visible="yes" active="no"/>
+<layer number="58" name="bCAD" color="11" fill="1" visible="yes" active="no"/>
 <layer number="90" name="Modules" color="5" fill="1" visible="yes" active="yes"/>
 <layer number="91" name="Nets" color="2" fill="1" visible="yes" active="yes"/>
@@
 <part name="R21" library="rcl" deviceset="R-EU_" device="R0805" value="15k"/>
 <part name="R22" library="rcl" deviceset="R-EU_" device="R0805" value="15k"/>
-<part name="U$2" library="adafruit" deviceset="SDMMC" device="06132"/>
+<part name="U$2" library="adafruit" deviceset="SDMMC" device="HALFHEIGHT" value="SDMMCHALFHEIGHT"/>
 <part name="GND10" library="supply1" deviceset="GND" device=""/>
 <part name="R23" library="rcl" deviceset="R-EU_" device="M0805" value="47K"/>
@@
 <part name="C30" library="rcl" deviceset="C-EU" device="C0805" value="0.1uF"/>
 <part name="GND17" library="supply1" deviceset="GND" device=""/>
-<part name="POW" library="Eagle_Wuerth_Elektronik_Switch_rev15b" deviceset="450302014072" device=""/>
+<part name="POW" library="Eagle_Wuerth_Elektronik_Switch_rev15b" deviceset="450302014072" device="ROCKER" value="450302014072ROCKER"/>
 <part name="R7" library="rcl" deviceset="R-EU_" device="R0805" value="4k7"/>
 <part name="C31" library="rcl" deviceset="C-EU" device="C0805" value="10uF"/>
@@
 <part name="H6" library="holes" deviceset="MOUNT-PAD-ROUND" device="2.5"/>
 <part name="GND19" library="supply1" deviceset="GND" device=""/>
+<part name="H7" library="holes" deviceset="MOUNT-PAD-ROUND" device="2.5"/>
 </parts>
 <sheets>
@@
 <wire x1="-7.62" y1="81.28" x2="-7.62" y2="63.5" width="0.1524" layer="91"/>
 <junction x="-7.62" y="33.02"/>
-<pinref part="POW" gate="G$1" pin="1"/>
 <wire x1="-7.62" y1="63.5" x2="-7.62" y2="50.8" width="0.1524" layer="91"/>
 <wire x1="-7.62" y1="50.8" x2="-7.62" y2="33.02" width="0.1524" layer="91"/>
-<wire x1="-22.86" y1="76.2" x2="-22.86" y2="63.5" width="0.1524" layer="91"/>
-<wire x1="-22.86" y1="63.5" x2="-7.62" y2="63.5" width="0.1524" layer="91"/>
 <junction x="-7.62" y="63.5"/>
 <pinref part="R30" gate="G$1" pin="1"/>
 <pinref part="R7" gate="G$1" pin="1"/>
+<wire x1="-12.7" y1="63.5" x2="-7.62" y2="63.5" width="0.1524" layer="91"/>
 <wire x1="0" y1="48.26" x2="0" y2="50.8" width="0.1524" layer="91"/>
 <wire x1="0" y1="50.8" x2="0" y2="53.34" width="0.1524" layer="91"/>
@@
 <junction x="0" y="50.8"/>
 <label x="-25.4" y="33.02" size="1.778" layer="95"/>
+<pinref part="POW" gate="G$1" pin="2"/>
+<wire x1="-12.7" y1="73.66" x2="-12.7" y2="63.5" width="0.1524" layer="91"/>
 </segment>
 </net>
@@
 <net name="N$139" class="0">
 <segment>
-<pinref part="POW" gate="G$1" pin="3"/>
-<wire x1="-12.7" y1="78.74" x2="-12.7" y2="88.9" width="0.1524" layer="91"/>
 <pinref part="PF1" gate="G$1" pin="2"/>
-<wire x1="-12.7" y1="88.9" x2="-25.4" y2="88.9" width="0.1524" layer="91"/>
+<wire x1="-22.86" y1="88.9" x2="-25.4" y2="88.9" width="0.1524" layer="91"/>
+<pinref part="POW" gate="G$1" pin="1"/>
+<wire x1="-22.86" y1="88.9" x2="-22.86" y2="76.2" width="0.1524" layer="91"/>
 </segment>
 </net>
@@
 <instance part="H6" gate="G$1" x="38.1" y="22.86"/>
 <instance part="GND19" gate="1" x="15.24" y="5.08"/>
+<instance part="H7" gate="G$1" x="38.1" y="12.7"/>
 </instances>
 <busses>
@@
 <wire x1="15.24" y1="7.62" x2="-33.02" y2="7.62" width="0.1524" layer="91"/>
 <junction x="15.24" y="7.62"/>
-<wire x1="15.24" y1="7.62" x2="15.24" y2="22.86" width="0.1524" layer="91"/>
+<wire x1="15.24" y1="7.62" x2="15.24" y2="12.7" width="0.1524" layer="91"/>
+<wire x1="15.24" y1="12.7" x2="15.24" y2="22.86" width="0.1524" layer="91"/>
 <wire x1="15.24" y1="22.86" x2="15.24" y2="48.26" width="0.1524" layer="91"/>
 <wire x1="15.24" y1="48.26" x2="15.24" y2="91.44" width="0.1524" layer="91"/>
@@
 <wire x1="35.56" y1="22.86" x2="15.24" y2="22.86" width="0.1524" layer="91"/>
 <junction x="15.24" y="22.86"/>
+<pinref part="H7" gate="G$1" pin="MOUNT"/>
+<wire x1="35.56" y1="12.7" x2="15.24" y2="12.7" width="0.1524" layer="91"/>
+<junction x="15.24" y="12.7"/>
 </segment>
 </net>

Commit message: HDMI port
git-svn-id: http://www.64kib.com/atarixlfpga_svn/trunk/atari_800xl@436 d6161ac3-aae1-4d52-9b05-ea9ac36b53d3
Parts:
- added RN28, RN29: 270, resistor-array:742-8742_3
- added X1: HDMI, raspberrypi_cm:HDMI
- POW: value 450302014072ROCKER -> 450302014072ROCKER2; device Eagle_Wuerth_Elektronik_Switch_rev15b:450302014072ROCKER -> Eagle_Wuerth_Elektronik_Switch_rev15b:450302014072ROCKER2
Connections:
- new net N$134: RN28.8, X1.TX2_P
- new net N$144: RN28.7, X1.TX2_N
- new net N$146: RN28.6, X1.TX1_P
- new net N$147: RN28.5, X1.TX1_N
- new net N$148: RN29.8, X1.TX0_P
- new net N$149: RN29.7, X1.TX0_N
- new net N$150: RN29.6, X1.CLK_P
- new net N$151: RN29.5, X1.CLK_N
- net 5V0: now also POW.3, X1.+5V; no longer POW.2
- net GND: now also X1.GND@1, X1.GND@2, X1.GND@3, X1.GND@4, X1.GND@5, X1.GND@6, X1.GND@7, X1.GND@8, X1.GND@9
- net VGA_B1: now also RN29.2
- net VGA_B4: now also RN29.1
- net VGA_B5: now also RN29.4
- net VGA_B6: now also RN29.3
- net VGA_R0: now also RN28.1
- net VGA_R1: now also RN28.2
- net VGA_R3: now also RN28.4
- net VGA_R4: now also RN28.3

Commit message: Update from Panos (many thanks). Adjusted labels, tidied endings where nets meet pins
git-svn-id: http://www.64kib.com/atarixlfpga_svn/trunk/atari_800xl@472 d6161ac3-aae1-4d52-9b05-ea9ac36b53d3
Parts:
- AUDIO: device stereoaudiojack:AUDIO-JACK2CUI -> LIBstereoaudiojack:AUDIO-JACK2CUI
- renumbered 5VIN to 5V_IN, 5VINB to 5V_IN_B, COMPOSITE to C-VIDEO, DAC to VIDEODACSA, GPIOA to GPIO_A, GPIOB to GPIO_B, GPIOC to GPIO_C, POW to POWER_SW, PS2 to PS/2, SVIDEO to S-VIDEO, U1 to SPI, USBA to USB.A, USBB to USB.B, X1 to HDMI
Other:
- moved on the sheet: AUDIO
