File: atari_chips/hardware/pokeymaxv4/pokeymax4.brd (EAGLE design)
At the start: 20.7 x 52.8 mm, 39 parts, among them CN1 18nF, U1 TSV854IQ4T, U2 SN74CB3T16211SM, U3 MAX10, U4 SN74CB3T16211SM, X1 ASE

Commit message: Renumbering left it called pokeymax1
git-svn-id: http://www.64kib.com/atarixlfpga_svn/trunk/atari_800xl@1391 d6161ac3-aae1-4d52-9b05-ea9ac36b53d3
Parts:
- renumbered POKEYMAX1 to POKEYMAX4
